File: hardware/badge/MZ2023.kicad_pcb (KiCad board)
At the start: 2 copper layers, 70 x 95.6 mm, 30 parts, among them J1 Conn_01x04, J10 SAO, J2 Conn_01x04, J3 Conn_01x04, J4 Conn_01x04, J5 Conn_01x14_Female, J6 Conn_01x04_Female, J8 Conn_01x04, J9 SAO, Q2 DMG2301L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

Commit message: PCB Layout
Parts:
- removed D8: WS2812B, LED_SMD:LED_WS2812B_PLCC4_5.0x5.0mm_P3.2mm
- removed J10, J9: SAO, Connector_PinSocket_2.54mm:PinSocket_2x03_P2.54mm_Vertical_SMD
- removed J8: Conn_01x04, Tillo:Grove_SMD
- removed U2: BD3571YFP, Package_TO_SOT_SMD:TO-252-2
- added C3: 10µ, Capacitor_SMD:C_1206_3216Metric_Pad1.33x1.80mm_HandSolder, F.Cu at (87.4, 58.5)
- added D10: D, Diode_SMD:D_MiniMELF, F.Cu at (81.3, 63.6)
- added R5: 1k, Resistor_SMD:R_0805_2012Metric_Pad1.20x1.40mm_HandSolder, F.Cu at (93.2, 62.0)
- added R6: 1k, Resistor_SMD:R_0805_2012Metric_Pad1.20x1.40mm_HandSolder, F.Cu at (92.2, 58.6)
- added SW4: SW_Push_SPDT, Button_Switch_THT:SW_CuK_OS102011MA1QN1_SPDT_Angled, B.Cu at (73.5, 76.0)
- added TP2: NP, TestPoint:TestPoint_Keystone_5015_Micro-Minature, B.Cu at (115.9, 57.7)
- added TP3: NP, TestPoint:TestPoint_Keystone_5015_Micro-Minature, B.Cu at (116.0, 54.4)
- added TP5: NP, TestPoint:TestPoint_Keystone_5015_Micro-Minature, B.Cu at (116.0, 48.0)
- added TP6: NP, TestPoint:TestPoint_Keystone_5015_Micro-Minature, B.Cu at (116.0, 44.8)
- added TP7: NP, TestPoint:TestPoint_Keystone_5015_Micro-Minature, B.Cu at (116.0, 41.5)
- added U3: MCP73831-2-OT, Package_TO_SOT_SMD:SOT-23-5, F.Cu at (90.2, 62.0)
- added kibuzzard-6368F1D8: G***, kibuzzard-6368F1D8, F.Cu at (70.6, 60.0)
- added kibuzzard-6368F201: G***, kibuzzard-6368F201, F.Cu at (70.5, 49.0)
- added kibuzzard-6368F224: G***, kibuzzard-6368F224, F.Cu at (137.5, 74.0)
- added kibuzzard-6368F2A8: G***, kibuzzard-6368F2A8, F.Cu at (83.5, 42.7)
- added kibuzzard-6368F2D1: G***, kibuzzard-6368F2D1, F.Cu at (81.5, 42.7)
- added kibuzzard-6368F305: G***, kibuzzard-6368F305, F.Cu at (91.7, 42.7)
- added kibuzzard-6368F322: G***, kibuzzard-6368F322, F.Cu at (93.7, 42.7)
- added kibuzzard-6368F378: G***, kibuzzard-6368F378, F.Cu at (100.4, 69.8)
- added kibuzzard-6368F386: G***, kibuzzard-6368F386, F.Cu at (98.4, 69.8)
- added kibuzzard-6368F3A3: G***, kibuzzard-6368F3A3, F.Cu at (86.5, 70.0)
- added kibuzzard-6368F3AE: G***, kibuzzard-6368F3AE, F.Cu at (84.5, 70.0)
- added kibuzzard-6368F490: G***, kibuzzard-6368F490, F.Cu at (136.3, 39.5)
- added kibuzzard-6368F495: G***, kibuzzard-6368F495, F.Cu at (135.3, 42.1)
- added kibuzzard-6368F4A2: G***, kibuzzard-6368F4A2, F.Cu at (136.1, 44.9)
- added kibuzzard-6368F4DE: G***, kibuzzard-6368F4DE, F.Cu at (135.0, 47.2)
- added kibuzzard-6368F4F7: G***, kibuzzard-6368F4F7, F.Cu at (136.5, 49.7)
- added kibuzzard-6368F503: G***, kibuzzard-6368F503, F.Cu at (135.0, 52.3)
- added kibuzzard-6368F536: G***, kibuzzard-6368F536, F.Cu at (140.5, 68.7)
- added kibuzzard-6368F610: G***, kibuzzard-6368F610, B.Cu at (90.0, 32.0)
- added kibuzzard-6369234D: G***, kibuzzard-6369234D, B.Cu at (92.0, 33.5)
- added kibuzzard-63692365: G***, kibuzzard-63692365, B.Cu at (90.0, 33.5)
- added kibuzzard-636923C0: G***, kibuzzard-636923C0, B.Cu at (71.5, 72.0)
- D7: value WS2812B -> BAT; footprint LED_SMD:LED_WS2812B_PLCC4_5.0x5.0mm_P3.2mm -> LED_SMD:LED_0603_1608Metric_Pad1.05x0.95mm_HandSolder
- J5: value Conn_01x14_Female -> Conn_01x08_Female; footprint Connector_PinSocket_2.54mm:PinSocket_1x14_P2.54mm_Vertical -> Connector_PinSocket_2.54mm:PinSocket_1x08_P2.54mm_Vertical_SMD_Pin1Right
- J6: value Conn_01x04_Female -> Conn_01x02_Male; footprint Connector_PinSocket_2.54mm:PinSocket_1x04_P2.54mm_Vertical -> Connector_JST:JST_PH_S2B-PH-K_1x02_P2.00mm_Horizontal; moved to B.Cu
- SW1, SW2, SW3: footprint Button_Switch_SMD:SW_SPST_Omron_B3FS-105xP -> Button_Switch_SMD:SW_Push_1P1T_NO_CK_KMR2
- TP1: renamed from TP5; moved to B.Cu
- TP4: moved to B.Cu
- moved SW2 115.5 mm to (67.6, 48.9), turned to -90 degrees
- moved SW1 107.3 mm to (67.6, 59.9), turned to -90 degrees
- moved J6 100.7 mm to (91.9, 36.0), turned to 180 degrees
- moved J3 95.9 mm to (98.5, 33.0)
- moved R4 82.5 mm to (104.0, 56.0), turned to 90 degrees
- moved J4 72.0 mm to (84.5, 33.0)
- moved R2 67.8 mm to (135.0, 55.5), turned to -90 degrees
- moved TP4 67.2 mm to (116.1, 51.3), turned to 180 degrees
- moved R3 65.2 mm to (137.5, 63.5), turned to 90 degrees
- moved TP1 64.3 mm to (124.9, 49.6), turned to 180 degrees
- moved U1 59.2 mm to (120.0, 56.0)
- moved D9 56.6 mm to (140.0, 63.5), turned to 90 degrees
- moved R1 56.1 mm to (135.0, 60.5), turned to 90 degrees
- moved Q2 56.1 mm to (85.9, 61.9)
- moved SW3 52.8 mm to (137.5, 77.0)
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Connections:
- D6 pad 2: Net-(D6-Pad2) -> unconnected-(D6-Pad2)
- D7 pad 1: VCC -> Net-(D7-Pad1)
- D7 pad 2: Net-(D7-Pad2) -> VBUS
- J5 pad 3: /GP11 -> /GP28
- J5 pad 7: /GP15 -> /GP11
- J5 pad 8: +3V3 -> /GP10
- J6 pad 1: unconnected-(J6-Pad1) -> +BATT
- J6 pad 2: unconnected-(J6-Pad2) -> GND
- Q2 pad 2: Net-(Q2-Pad2) -> +BATT
- R3 pad 1: /GP16 -> /GP8
- TP4 pad 1: Net-(TP4-Pad1) -> /GP19
- U1 pad 11: Net-(TP4-Pad1) -> /GP8
- U1 pad 39: VCC -> Net-(U1-Pad39)
Routing:
- net /GP6: track 0.00 -> 75.4 mm
- net /GP7: track 0.00 -> 74.3 mm
- net /GP4: track 0.00 -> 73.4 mm, vias 0 -> 2
- net /GP5: track 0.00 -> 72.6 mm, vias 0 -> 2
- net /NPXL: track 0.00 -> 55.9 mm, vias 0 -> 2
- net /RST: track 0.00 -> 55.2 mm, vias 0 -> 2
- net /GP3: track 0.00 -> 48.2 mm, vias 0 -> 2
- net /GP2: track 0.00 -> 48.0 mm
- net VBUS: track 0.00 -> 46.8 mm, vias 0 -> 3
- net Net-(U1-Pad39): track 0.00 -> 41.5 mm, vias 0 -> 1
- net /GP28: track 0.00 -> 39.5 mm, vias 0 -> 2
- net /GP0: track 0.00 -> 38.8 mm
- net /GP27: track 0.00 -> 36.9 mm, vias 0 -> 2
- net /GP26: track 0.00 -> 31.5 mm, vias 0 -> 2
- net /GP1: track 0.00 -> 30.0 mm
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- added copper zone on B.Cu, net +3V3
- added copper zone on F.Cu, net GND
- added copper zone on B.Cu, net VCC
Other:
- board size 70 x 95.6 mm -> 77 x 51.3 mm
