File: hardware/badge/MZ2023.kicad_pcb (KiCad board)
At the start: 2 copper layers, 77 x 51.4 mm, 88 parts, among them J1 Conn_01x04, J2 Conn_01x04, J3 Conn_01x04, J4 Conn_01x04, J5 Conn_01x10_Female, J6 Conn_01x02_Male, J7 Conn_01x05_Female, J8 Conn_Coaxial, J9 Conn_02x03_Counter_Clockwise, Q2 DMG2301L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

Commit message: badge: improving bottomo slick
Parts:
- added kibuzzard-6464F92F: G***, kibuzzard-6464F92F, B.Cu at (122.8, 80.2)
- added kibuzzard-6464F984: G***, kibuzzard-6464F984, B.Cu at (122.8, 93.5)
- added kibuzzard-6464F9A8: G***, kibuzzard-6464F9A8, B.Cu at (131.4, 86.8)
