File: hardware/badge/MZ2023-rounded.kicad_pcb (KiCad board)
At the start: 2 copper layers, 77 x 51.3 mm, 59 parts, among them J1 Conn_01x04, J2 Conn_01x04, J3 Conn_01x04, J4 Conn_01x04, J5 Conn_01x08_Female, J6 Conn_01x02_Male, J7 Conn_01x07_Female, Q2 DMG2301L, SW1 SW_Push, SW2 SW_Push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

Commit message: prototype
Parts:
- moved kibuzzard-6368F610 36.0 mm to (122.6, 74.1), turned to 180 degrees
- moved kibuzzard-6369234D 18.9 mm to (124.6, 75.6)
- moved kibuzzard-63692365 17.0 mm to (122.6, 75.6)
- moved kibuzzard-6370DC53 1.27 mm to (116.2, 82.3)
- moved kibuzzard-6370DC69 1.27 mm to (114.0, 82.3)
- moved R1 0.60 mm to (139.1, 104.2)
- moved R2 0.16 mm to (138.8, 99.0)
Routing:
- net /GP6: track 70.1 -> 67.6 mm
- net /GP17: track 52.7 -> 54.9 mm
- net /GP5: track 83.2 -> 81.0 mm
- net /GP0: track 39.2 -> 37.8 mm
- net /GP3: track 50.5 -> 49.2 mm
- net /NPXL: track 44.6 -> 43.5 mm
- net /GP9: track 68.7 -> 67.6 mm
- net /GP19: track 53.3 -> 52.3 mm
- net /GP2: track 50.4 -> 49.6 mm
- net /GP7: track 75.4 -> 74.6 mm
- net VCC: track 21.5 -> 20.8 mm
- net /GP21: track 52.7 -> 52.0 mm
- net /GP4: track 78.1 -> 77.4 mm
- net Net-(SW4-Pad2): track 44.4 -> 43.8 mm
- net VBUS: track 50.3 -> 49.7 mm
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