File: hardware/badge/MZ2023.kicad_sch (KiCad schematic)
At the start: 45 parts, among them J1 Conn_01x04, J2 Conn_01x04, J3 Conn_01x04, J4 Conn_01x04, J5 Conn_01x10_Female, J6 Conn_01x02_Male, J7 Conn_01x05_Female, J8 Conn_Coaxial, J9 Conn_02x03_Counter_Clockwise, Q2 DMG2301L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

Commit message: adding component Mouser/Digikey part numbers to schematic. Generating ibom
Parts:
- C1: Mouser (none) -> 187-CL21A475KPFNNNG
- C2, C4, J8, J9, TP1: DNP (none) -> yes
- C3: Mouser (none) -> 187-CL31A106MAHNNNE
- D1, D2, D3, D4, D5, D6: Digikey (none) -> 1528-1542-ND; Mouser (none) -> 485-2659
- D11, D12, D7, D8, D9: Mouser (none) -> 710-150060VS75000
- J5: Mouser (none) -> 649-1012937891001BLF
- J7: Mouser (none) -> 649-1012937890503BLF
- L1: Mouser (none) -> 603-RC0805FR-070RL
- R1, R4: Mouser (none) -> 603-RT0603FRE1310KL
- R10, R11, R12, R3, R5, R6, R9: Mouser (none) -> 603-RT0603DRE071KL
- R7, R8: Mouser (none) -> 603-RT0603FRE0722RL
Changed lines of the file:
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@@
+      (effects (font (size 1.27 1.27)) hide)
+    )
+    (property "Mouser" " 710-150060VS75000 " (at 118.11 154.94 90)
+      (effects (font (size 1.27 1.27)) hide)
+    )
+    (property "Digikey" "" (at 118.11 154.94 90)
       (effects (font (size 1.27 1.27)) hide)
     )
@@
       (effects (font (size 1.27 1.27)) hide)
     )
+    (property "Mouser" "603-RT0603DRE071KL" (at 117.475 53.34 90)
+      (effects (font (size 1.27 1.27)) hide)
+    )
     (pin "1")
     (pin "2")
@@
       (effects (font (size 1.27 1.27)) hide)
     )
+    (property "Mouser" "603-RT0603DRE071KL" (at 266.7 82.55 0)
+      (effects (font (size 1.27 1.27)) hide)
+    )
     (pin "1")
     (pin "2")
@@
     )
     (property "Datasheet" "~" (at 266.065 31.75 0)
+      (effects (font (size 1.27 1.27)) hide)
+    )
+    (property "Mouser" "603-RT0603FRE1310KL" (at 266.065 31.75 0)
       (effects (font (size 1.27 1.27)) hide)
     )
@@
       (effects (font (size 1.27 1.27)) (justify left top) hide)
     )
+    (property "Mouser" "485-2659" (at 225.425 118.745 0)
+      (effects (font (size 1.27 1.27)) hide)
+    )
+    (property "Digikey" "1528-1542-ND" (at 225.425 118.745 0)
+      (effects (font (size 1.27 1.27)) hide)
+    )
     (pin "1")
     (pin "2")
@@
       (effects (font (size 1.27 1.27)) (justify left top) hide)
     )
+    (property "Mouser" "485-2659" (at 154.305 118.745 0)
+      (effects (font (size 1.27 1.27)) hide)
+    )
+    (property "Digikey" "1528-1542-ND" (at 154.305 118.745 0)
+      (effects (font (size 1.27 1.27)) hide)
+    )
     (pin "1")
     (pin "2")
@@
     )
     (property "Datasheet" "~" (at 98.425 108.585 0)
+      (effects (font (size 1.27 1.27)) hide)
+    )
+    (property "Mouser" "649-1012937890503BLF" (at 98.425 108.585 0)
       (effects (font (size 1.27 1.27)) hide)
     )
@@
     (property "Datasheet" "https://cdn-shop.adafruit.com/product-files/2686/SK6812MINI_REV.01-1-2.pdf" (at 192.405 128.27 0)
       (effects (font (size 1.27 1.27)) (justify left top) hide)
+    )
+    (property "Mouser" "485-2659" (at 189.865 118.745 0)
+      (effects (font (size 1.27 1.27)) hide)
+    )
+    (property "Digikey" "1528-1542-ND" (at 189.865 118.745 0)
+      (effects (font (size 1.27 1.27)) hide)
     )
     (pin "1")
@@
       (effects (font (size 1.27 1.27)) (justify left top) hide)
     )
+    (property "Mouser" "485-2659" (at 172.085 118.745 0)
+      (effects (font (size 1.27 1.27)) hide)
+    )
+    (property "Digikey" "1528-1542-ND" (at 172.085 118.745 0)
+      (effects (font (size 1.27 1.27)) hide)
+    )
     (pin "1")
     (pin "2")
@@
       (effects (font (size 1.27 1.27)) hide)
     )
+    (property "Mouser" "603-RT0603DRE071KL" (at 142.875 55.245 90)
+      (effects (font (size 1.27 1.27)) hide)
+    )
     (pin "1")
     (pin "2")
@@
     )
     (property "Datasheet" " ~" (at 133.35 172.72 0)
+      (effects (font (size 1.27 1.27)) hide)
+    )
+    (property "DNP" "yes" (at 133.35 172.72 0)
       (effects (font (size 1.27 1.27)) hide)
     )
@@
       (effects (font (size 1.27 1.27)) hide)
     )
+    (property "Mouser" " 710-150060VS75000 " (at 46.355 166.37 90)
+      (effects (font (size 1.27 1.27)) hide)
+    )
+    (property "Digikey" "" (at 46.355 166.37 90)
+      (effects (font (size 1.27 1.27)) hide)
+    )
     (pin "1")
     (pin "2")
@@
       (effects (font (size 1.27 1.27)) hide)
     )
+    (property "Mouser" "603-RT0603FRE0722RL" (at 67.945 187.325 90)
+      (effects (font (size 1.27 1.27)) hide)
+    )
     (pin "1")
     (pin "2")
@@
     )
     (property "Datasheet" "~" (at 158.115 49.53 0)
+      (effects (font (size 1.27 1.27)) hide)
+    )
+    (property "Mouser" " 187-CL31A106MAHNNNE " (at 158.115 49.53 0)
       (effects (font (size 1.27 1.27)) hide)
     )
@@
       (effects (font (size 1.27 1.27)) hide)
     )
+    (property "Mouser" " 710-150060VS75000 " (at 266.7 93.345 90)
+      (effects (font (size 1.27 1.27)) hide)
+    )
+    (property "Digikey" "" (at 266.7 93.345 90)
+      (effects (font (size 1.27 1.27)) hide)
+    )
     (pin "1")
     (pin "2")
@@
       (effects (font (size 1.27 1.27)) hide)
     )
+    (property "Mouser" "603-RT0603DRE071KL" (at 46.355 175.895 0)
+      (effects (font (size 1.27 1.27)) hide)
+    )
     (pin "1")
     (pin "2")
@@
       (effects (font (size 1.27 1.27)) hide)
     )
+    (property "DNP" "yes" (at 118.745 179.705 0)
+      (effects (font (size 1.27 1.27)) hide)
+    )
     (pin "1")
     (pin "2")
@@
     )
     (property "Datasheet" "~" (at 111.76 172.72 0)
+      (effects (font (size 1.27 1.27)) hide)
+    )
+    (property "Mouser" "603-RC0805FR-070RL" (at 111.76 172.72 90)
       (effects (font (size 1.27 1.27)) hide)
     )
@@
       (effects (font (size 1.27 1.27)) hide)
     )
+    (property "DNP" "yes" (at 104.775 179.705 0)
+      (effects (font (size 1.27 1.27)) hide)
+    )
     (pin "1")
     (pin "2")
@@
     )
     (property "Datasheet" "~" (at 108.585 154.94 0)
+      (effects (font (size 1.27 1.27)) hide)
+    )
+    (property "Mouser" "603-RT0603DRE071KL" (at 108.585 154.94 0)
       (effects (font (size 1.27 1.27)) hide)
     )
@@
     )
     (property "Datasheet" "~" (at 38.1 166.37 0)
+      (effects (font (size 1.27 1.27)) hide)
+    )
+    (property "Mouser" " 710-150060VS75000 " (at 38.1 166.37 90)
+      (effects (font (size 1.27 1.27)) hide)
+    )
+    (property "Digikey" "" (at 38.1 166.37 90)
       (effects (font (size 1.27 1.27)) hide)
     )
@@
       (effects (font (size 1.27 1.27)) hide)
     )
+    (property "Mouser" "603-RT0603FRE1310KL" (at 186.055 56.515 0)
+      (effects (font (size 1.27 1.27)) hide)
+    )
     (pin "1")
     (pin "2")
@@
       (effects (font (size 1.27 1.27)) hide)
     )
+    (property "Mouser" "187-CL21A475KPFNNNG" (at 56.515 151.765 0)
+      (effects (font (size 1.27 1.27)) hide)
+    )
     (pin "1")
     (pin "2")
@@
       (effects (font (size 1.27 1.27)) hide)
     )
+    (property "Mouser" "603-RT0603DRE071KL" (at 38.1 175.895 0)
+      (effects (font (size 1.27 1.27)) hide)
+    )
     (pin "1")
     (pin "2")
@@
     )
     (property "Datasheet" "~" (at 48.26 113.665 0)
+      (effects (font (size 1.27 1.27)) hide)
+    )
+    (property "Mouser" "649-1012937891001BLF" (at 48.26 113.665 0)
       (effects (font (size 1.27 1.27)) hide)
     )
@@
       (effects (font (size 1.27 1.27)) hide)
     )
+    (property "Mouser" "603-RT0603FRE0722RL" (at 67.945 182.88 90)
+      (effects (font (size 1.27 1.27)) hide)
+    )
     (pin "1")
     (pin "2")
@@
       (effects (font (size 1.27 1.27)) (justify left top) hide)
     )
+    (property "Mouser" "485-2659" (at 136.525 118.745 0)
+      (effects (font (size 1.27 1.27)) hide)
+    )
+    (property "Digikey" "1528-1542-ND" (at 136.525 118.745 0)
+      (effects (font (size 1.27 1.27)) hide)
+    )
     (pin "1")
     (pin "2")
@@
       (effects (font (size 1.27 1.27)) hide)
     )
+    (property "Mouser" "603-RT0603DRE071KL" (at 117.475 62.865 90)
+      (effects (font (size 1.27 1.27)) hide)
+    )
     (pin "1")
     (pin "2")
@@
       (effects (font (size 1.27 1.27)) hide)
     )
+    (property "DNP" "yes" (at 125.095 172.72 0)
+      (effects (font (size 1.27 1.27)) hide)
+    )
     (pin "1")
     (instances
@@
       (effects (font (size 1.27 1.27)) hide)
     )
+    (property "Mouser" " 710-150060VS75000 " (at 149.86 54.61 90)
+      (effects (font (size 1.27 1.27)) hide)
+    )
+    (property "Digikey" "" (at 149.86 54.61 90)
+      (effects (font (size 1.27 1.27)) hide)
+    )
     (pin "1")
     (pin "2")
@@
       (effects (font (size 1.27 1.27)) (justify left top) hide)
     )
+    (property "Mouser" "485-2659" (at 207.645 118.745 0)
+      (effects (font (size 1.27 1.27)) hide)
+    )
+    (property "Digikey" "1528-1542-ND" (at 207.645 118.745 0)
+      (effects (font (size 1.27 1.27)) hide)
+    )
     (pin "1")
     (pin "2")
@@
       (effects (font (size 1.27 1.27)) hide)
     )
+    (property "DNP" "yes" (at 150.495 150.495 0)
+      (effects (font (size 1.27 1.27)) hide)
+    )

Commit message: parts numbers: completing digikey
Parts:
- C1: Digikey (none) -> 1276-6464-1-ND
- C3: Digikey (none) -> 1276-1181-1-ND
- D11, D12, D7, D8, D9: Digikey (none) -> 732-4980-1-ND
- J5: Digikey (none) -> 10129378-910002BLF-ND
- J7: Digikey (none) -> 664-G800W303018EU-ND
- L1: Digikey (none) -> 311-0.0CRCT-ND
- Q2: Digikey (none) -> DMG2301L-7DICT-ND; Digitec DMG2301L-7DICT-ND -> (none)
- R1, R4: Digikey (none) -> 13-RT0603FRE1310KLCT-ND
- R10, R11, R12, R3, R5, R6, R9: Digikey (none) -> 311-2475-1-ND
- R7, R8: Digikey (none) -> YAG5950CT-ND
Changed lines of the file:
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@@
       (effects (font (size 1.27 1.27)) hide)
     )
-    (property "Digikey" "" (at 118.11 154.94 90)
+    (property "Digikey" "732-4980-1-ND" (at 118.11 154.94 90)
       (effects (font (size 1.27 1.27)) hide)
     )
@@
       (effects (font (size 1.27 1.27)) hide)
     )
+    (property "Digikey" "311-2475-1-ND" (at 117.475 53.34 90)
+      (effects (font (size 1.27 1.27)) hide)
+    )
     (pin "1")
     (pin "2")
@@
       (effects (font (size 1.27 1.27)) hide)
     )
+    (property "Digikey" "311-2475-1-ND" (at 266.7 82.55 0)
+      (effects (font (size 1.27 1.27)) hide)
+    )
     (pin "1")
     (pin "2")
@@
     )
     (property "Mouser" "603-RT0603FRE1310KL" (at 266.065 31.75 0)
+      (effects (font (size 1.27 1.27)) hide)
+    )
+    (property "Digikey" "13-RT0603FRE1310KLCT-ND" (at 266.065 31.75 0)
       (effects (font (size 1.27 1.27)) hide)
     )
@@
     )
     (property "Mouser" "649-1012937890503BLF" (at 98.425 108.585 0)
+      (effects (font (size 1.27 1.27)) hide)
+    )
+    (property "Digikey" "664-G800W303018EU-ND" (at 98.425 108.585 0)
       (effects (font (size 1.27 1.27)) hide)
     )
@@
       (effects (font (size 1.27 1.27)) hide)
     )
+    (property "Digikey" "311-2475-1-ND" (at 142.875 55.245 90)
+      (effects (font (size 1.27 1.27)) hide)
+    )
     (pin "1")
     (pin "2")
@@
       (effects (font (size 1.27 1.27)) hide)
     )
-    (property "Digikey" "" (at 46.355 166.37 90)
+    (property "Digikey" "732-4980-1-ND" (at 46.355 166.37 90)
       (effects (font (size 1.27 1.27)) hide)
     )
@@
       (effects (font (size 1.27 1.27)) hide)
     )
+    (property "Digikey" "YAG5950CT-ND" (at 67.945 187.325 90)
+      (effects (font (size 1.27 1.27)) hide)
+    )
     (pin "1")
     (pin "2")
@@
     )
     (property "Mouser" " 187-CL31A106MAHNNNE " (at 158.115 49.53 0)
+      (effects (font (size 1.27 1.27)) hide)
+    )
+    (property "Digikey" "1276-1181-1-ND" (at 158.115 49.53 0)
       (effects (font (size 1.27 1.27)) hide)
     )
@@
       (effects (font (size 1.27 1.27)) hide)
     )
-    (property "Digikey" "" (at 266.7 93.345 90)
+    (property "Digikey" "732-4980-1-ND" (at 266.7 93.345 90)
       (effects (font (size 1.27 1.27)) hide)
     )
@@
       (effects (font (size 1.27 1.27)) hide)
     )
+    (property "Digikey" "311-2475-1-ND" (at 46.355 175.895 0)
+      (effects (font (size 1.27 1.27)) hide)
+    )
     (pin "1")
     (pin "2")
@@
     )
     (property "Mouser" "603-RC0805FR-070RL" (at 111.76 172.72 90)
+      (effects (font (size 1.27 1.27)) hide)
+    )
+    (property "Digikey" "311-0.0CRCT-ND" (at 111.76 172.72 90)
       (effects (font (size 1.27 1.27)) hide)
     )
@@
       (effects (font (size 1.27 1.27)) hide)
     )
+    (property "Digikey" "311-2475-1-ND" (at 108.585 154.94 0)
+      (effects (font (size 1.27 1.27)) hide)
+    )
     (pin "1")
     (pin "2")
@@
       (effects (font (size 1.27 1.27)) hide)
     )
-    (property "Digikey" "" (at 38.1 166.37 90)
+    (property "Digikey" "732-4980-1-ND" (at 38.1 166.37 90)
       (effects (font (size 1.27 1.27)) hide)
     )
@@
       (effects (font (size 1.27 1.27)) hide)
     )
+    (property "Digikey" "13-RT0603FRE1310KLCT-ND" (at 186.055 56.515 0)
+      (effects (font (size 1.27 1.27)) hide)
+    )
     (pin "1")
     (pin "2")
@@
       (effects (font (size 1.27 1.27)) hide)
     )
+    (property "Digikey" "1276-6464-1-ND" (at 56.515 151.765 0)
+      (effects (font (size 1.27 1.27)) hide)
+    )
     (pin "1")
     (pin "2")
@@
       (effects (font (size 1.27 1.27)) hide)
     )
+    (property "Digikey" "311-2475-1-ND" (at 38.1 175.895 0)
+      (effects (font (size 1.27 1.27)) hide)
+    )
     (pin "1")
     (pin "2")
@@
     )
     (property "Mouser" "649-1012937891001BLF" (at 48.26 113.665 0)
+      (effects (font (size 1.27 1.27)) hide)
+    )
+    (property "Digikey" "10129378-910002BLF-ND" (at 48.26 113.665 0)
       (effects (font (size 1.27 1.27)) hide)
     )
@@
       (effects (font (size 1.27 1.27)) hide)
     )
+    (property "Digikey" "YAG5950CT-ND" (at 67.945 182.88 90)
+      (effects (font (size 1.27 1.27)) hide)
+    )
     (pin "1")
     (pin "2")
@@
       (effects (font (size 1.27 1.27)) hide)
     )
+    (property "Digikey" "311-2475-1-ND" (at 117.475 62.865 90)
+      (effects (font (size 1.27 1.27)) hide)
+    )
     (pin "1")
     (pin "2")
@@
       (effects (font (size 1.27 1.27)) hide)
     )
-    (property "Digitec" "DMG2301L-7DICT-ND" (at 168.91 40.64 90)
+    (property "Digikey" "DMG2301L-7DICT-ND" (at 168.91 40.64 90)
       (effects (font (size 1.27 1.27)) hide)
     )
@@
       (effects (font (size 1.27 1.27)) hide)
     )
-    (property "Digikey" "" (at 149.86 54.61 90)
-      (effects (font (size 1.27 1.27)) hide)
-    )
+    (property "Digikey" "732-4980-1-ND" (at 149.86 54.61 90)
+      (effects (font (size 1.27 1.27)) hide)
+    )
