File: hardware/cover/cover.kicad_sch (KiCad schematic)
At the start: 9 parts, among them J1 Conn_01x05_Socket, J2 Conn_01x10_Socket, J3 Conn_02x03_Counter_Clockwise, J4 Conn_01x01, J5 Conn_01x01, J6 Conn_01x01, J7 Conn_01x01, J8 Conn_01x05_Socket, J9 Conn_01x10_Socket

Commit message: cover: adding PDFs schematic & layout
Other:
- note added: "Double footprint to allow left and right 1st pinof SMD pin headers"
- note added: "Pads for touch pads"
- note added: "SAO header"
- note added: "SAO header specs: https://hackaday.com/2019/03/20/introducing-the-shitty-add-on-v1-69bis-standard/"
- title: (none) -> MakeZurich 2023 name tag cover
Changed lines of the file:
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@@
 (kicad_sch (version 20230121) (generator eeschema)
   (paper "A4")
+  (title_block
+    (title "MakeZurich 2023 name tag cover")
+    (date "2023-06-03")
+    (rev "1")
+  )
   (junction (at 96.52 81.28) (diameter 0) (color 0 0 0 0)
   )
@@
     (stroke (width 0) (type default))
   )
+  (polyline (pts (xy 206.375 144.145) (xy 148.59 144.145))
+    (stroke (width 0) (type dot))
+  )
   (wire (pts (xy 96.52 81.28) (xy 96.52 101.6))
     (stroke (width 0) (type default))
   )
+  (polyline (pts (xy 89.535 73.66) (xy 89.535 116.84))
+    (stroke (width 0) (type dot))
+  )
   (wire (pts (xy 162.56 63.5) (xy 162.56 68.58))
     (stroke (width 0) (type default))
@@
     (stroke (width 0) (type default))
   )
+  (polyline (pts (xy 173.355 69.215) (xy 206.375 69.215))
+    (stroke (width 0) (type dot))
+  )
+  (polyline (pts (xy 173.355 69.215) (xy 173.355 77.47))
+    (stroke (width 0) (type dot))
+  )
   (wire (pts (xy 96.52 35.56) (xy 96.52 81.28))
     (stroke (width 0) (type default))
   )
+  (polyline (pts (xy 206.375 69.215) (xy 206.375 144.145))
+    (stroke (width 0) (type dot))
+  )
   (wire (pts (xy 175.26 137.16) (xy 185.42 137.16))
     (stroke (width 0) (type default))
   )
+  (polyline (pts (xy 89.535 73.66) (xy 137.16 73.66))
+    (stroke (width 0) (type dot))
+  )
   (wire (pts (xy 175.26 93.98) (xy 200.66 93.98))
     (stroke (width 0) (type default))
@@
     (stroke (width 0) (type default))
   )
+  (polyline (pts (xy 148.59 144.145) (xy 148.59 77.47))
+    (stroke (width 0) (type dot))
+  )
   (wire (pts (xy 93.98 91.44) (xy 93.98 111.76))
     (stroke (width 0) (type default))
   )
+  (polyline (pts (xy 137.16 73.66) (xy 137.16 116.84))
+    (stroke (width 0) (type dot))
+  )
   (wire (pts (xy 93.98 91.44) (xy 109.22 91.44))
     (stroke (width 0) (type default))
@@
     (stroke (width 0) (type default))
   )
+  (polyline (pts (xy 148.59 77.47) (xy 173.355 77.47))
+    (stroke (width 0) (type dot))
+  )
   (wire (pts (xy 175.26 129.54) (xy 200.66 129.54))
     (stroke (width 0) (type default))
@@
     (stroke (width 0) (type default))
   )
+  (polyline (pts (xy 137.16 116.84) (xy 89.535 116.84))
+    (stroke (width 0) (type dot))
+  )
   (wire (pts (xy 167.64 45.72) (xy 167.64 50.8))
     (stroke (width 0) (type default))
   )
+  (text "Double footprint to allow left and right \n1st pinof SMD pin headers"
+    (at 91.44 134.62 0)
+    (effects (font (size 1.27 1.27) (thickness 0.254) bold) (justify left bottom))
+  )
+  (text "SAO header" (at 147.955 58.42 0)
+    (effects (font (size 1.27 1.27) bold) (justify left bottom))
+  )
+  (text "SAO header specs:\nhttps://hackaday.com/2019/03/20/introducing-the-shitty-add-on-v1-69bis-standard/"
+    (at 177.8 164.465 0)
+    (effects (font (size 1.27 1.27) bold) (justify left bottom))
+  )
+  (text "Pads for touch pads" (at 132.715 32.385 0)
+    (effects (font (size 1.27 1.27) (thickness 0.254) bold) (justify left bottom))
+  )
   (label "SCL" (at 185.42 91.44 180) (fields_autoplaced)
